File: caterpillar.kicad_sch (KiCad schematic)
At the start: 32 parts, among them J1 Conn_ARM_JTAG_SWD_10, J2 SM02B-SRSS-TB_LF__SN_, J3 Castellated_2PTH_P1.27mm, J4 Castellated_2PTH_P1.27mm, M2 *, U1 STBB1-APUR, U2 ASM330LHHTR, U3 DRV8212P, U4 ADP2503ACPZ-3.3-R7, U6 max5419leta+T

Commit message: sch: add blue status LED on P0.01 (D1 + R1 470R, 0603)
P0.01 (module pin 35) -> R1 470R -> D1 anode, cathode -> GND;
active-high, ~0.7-0.9mA at blue Vf - fine for nRF standard drive.
Symbols/footprints from KiCad official libs (Device:LED imported
into lib_symbols, R reuses Device:R_Small_US; LED_0603/R_0603).
Netlist-verified including LED polarity (first draft had A/K
swapped by a cloned-template rotation - caught by netlist check).
BOM regenerated; README pin map updated.

Board side still pending: place D1/R1, route STATUS_LED (F8 first).
Parts:
- added D1: LED_BLUE, LED_SMD:LED_0603_1608Metric, symbol Device:LED
- added R1: 470, Resistor_SMD:R_0603_1608Metric, symbol Device:R_Small_US
Connections:
- net GND: now also D1.1 (K)
- net STATUS_LED: now reaches M2.35 (P0.01)
- net STATUS_LED: now also R1.2
- new net: D1.2 (A), R1.1
